File: PCB/Eagle 1.0/servoventil.brd (EAGLE design)
At the start: 58.8 x 51.2 mm, 34 parts, among them J1 ICSP 2x5, J2 SERIAL, J3 SERVO, J4 I2C, K1 ARK500/2, SW1 SPST_TACT-EVQQ2, T1 DMP2100U SOT23, T2 IRF7416PBF SO8, T3 FDV303N SOT23, T4 FDV303N SOT23

Commit message: Přidáno schéma
Parts:
- D2: value STTH4R02S DO214AB -> STTH4R02U DO214AA
- R2: value 10k 1203 -> 10k 1206
Changed lines of the file:
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@@
 <?xml version="1.0" encoding="utf-8"?>
 <!DOCTYPE eagle SYSTEM "eagle.dtd">
-<eagle version="9.2.2">
+<eagle version="9.3.0">
 <drawing>
 <settings>
@@
 <attribute name="VALUE" x="61.585409375" y="38.466209375" size="1.27" layer="28" rot="MR0"/>
 </element>
-<element name="D2" library="diode" library_urn="urn:adsk.eagle:library:210" package="DO214AA" package3d_urn="urn:adsk.eagle:package:43433/2" value="STTH4R02S  DO214AB" x="62.508728125" y="35.643034375" smashed="yes" rot="MR270">
+<element name="D2" library="diode" library_urn="urn:adsk.eagle:library:210" package="DO214AA" package3d_urn="urn:adsk.eagle:package:43433/2" value="STTH4R02U  DO214AA" x="62.508728125" y="35.643034375" smashed="yes" rot="MR270">
 <attribute name="NAME" x="63.07675" y="31.915190625" size="1.27" layer="26" ratio="10" rot="MR270"/>
 <attribute name="VALUE" x="70.294728125" y="52.253034375" size="1.27" layer="28" ratio="10" rot="MR270"/>
@@
 <attribute name="VALUE" x="89.530440625" y="57.054934375" size="1.27" layer="28" rot="MR270"/>
 </element>
-<element name="R2" library="rcl" library_urn="urn:adsk.eagle:library:334" package="R1206" package3d_urn="urn:adsk.eagle:package:23540/2" value="10k 1203" x="62.828553125" y="40.97374375" smashed="yes" rot="R270">
+<element name="R2" library="rcl" library_urn="urn:adsk.eagle:library:334" package="R1206" package3d_urn="urn:adsk.eagle:package:23540/2" value="10k 1206" x="62.828553125" y="40.97374375" smashed="yes" rot="R270">
 <attribute name="NAME" x="64.098553125" y="43.13549375" size="1.27" layer="25" font="vector" rot="R270"/>
 <attribute name="SPICEPREFIX" value="R" x="62.828553125" y="40.97374375" size="1.778" layer="27" rot="R270" display="off"/>
