File: PCB/Eagle 1.0/servoventil.sch (EAGLE design)
At the start: 34 parts, among them J1 ICSP 2x5, J2 SERIAL, J3 SERVO, J4 I2C, K1 ARK500/2, SW1 SPST_TACT-EVQQ2, T1 DMP2100U SOT23, T2 IRF7416PBF SO8, T3 FDV303N SOT23, T4 FDV303N SOT23

Commit message: Přidáno schéma
Parts:
- D2: value STTH4R02S DO214AB -> STTH4R02U DO214AA
- R2: value 10k 1203 -> 10k 1206
Changed lines of the file:
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@@
 <?xml version="1.0" encoding="utf-8"?>
 <!DOCTYPE eagle SYSTEM "eagle.dtd">
-<eagle version="9.2.2">
+<eagle version="9.3.0">
 <drawing>
 <settings>
@@
 <part name="IO1" library="bt_avr" deviceset="ATTINY1634" device="-SU" value="ATTINY1634 SO20W"/>
 <part name="F1" library="adafruit" library_urn="urn:adsk.eagle:library:420" deviceset="PTCFUSE" device="-1206" package3d_urn="urn:adsk.eagle:package:6240569/1" value="3,5A 1206"/>
-<part name="D2" library="diode" library_urn="urn:adsk.eagle:library:210" deviceset="DIODE-" device="DO214AA" package3d_urn="urn:adsk.eagle:package:43433/2" value="STTH4R02S  DO214AB"/>
+<part name="D2" library="diode" library_urn="urn:adsk.eagle:library:210" deviceset="DIODE-" device="DO214AA" package3d_urn="urn:adsk.eagle:package:43433/2" value="STTH4R02U  DO214AA"/>
 <part name="C1" library="rcl" library_urn="urn:adsk.eagle:library:334" deviceset="C-EU" device="C1206" package3d_urn="urn:adsk.eagle:package:23618/2" value="470n 1206"/>
 <part name="C2" library="rcl" library_urn="urn:adsk.eagle:library:334" deviceset="C-EU" device="C1206" package3d_urn="urn:adsk.eagle:package:23618/2" value="100n 1206"/>
 <part name="R1" library="rcl" library_urn="urn:adsk.eagle:library:334" deviceset="R-EU_" device="R1206" package3d_urn="urn:adsk.eagle:package:23540/2" value="10k 1206"/>
-<part name="R2" library="rcl" library_urn="urn:adsk.eagle:library:334" deviceset="R-EU_" device="R1206" package3d_urn="urn:adsk.eagle:package:23540/2" value="10k 1203"/>
+<part name="R2" library="rcl" library_urn="urn:adsk.eagle:library:334" deviceset="R-EU_" device="R1206" package3d_urn="urn:adsk.eagle:package:23540/2" value="10k 1206"/>
 <part name="J2" library="#PaJa_konektory" deviceset="S1G5_JUMP" device="" value="SERIAL"/>
 <part name="K1" library="#PaJa_konektory" deviceset="ARK500/2" device=""/>
